Commit message: explored urdf file's link and joint

File: robot/urdf/101.urdf (robot description, URDF)
Before this commit: robot myfirst, 1 links, 0 joints
Links:
- added link sub_link, mass 0.25; collision cylinder length=1 radius=0.1; visual cylinder length=1 radius=0.1
- link base_link: mass None -> 0.25; geometry collision cylinder length=0.6 radius=0.25; visual cylinder length=0.6 radius=0.25
Joints:
- added joint base_to_sub: type fixed, parent base_link, child sub_link, origin xyz=0.5 0 0 rpy=0 0 0, axis 1 0 0, limit lower=10 upper=0 effort=10 velocity=1
