Commit message: done with eval population without threading

File: temp.urdf (robot description, URDF)
Before this commit: robot jiejie, 13 links, 12 joints
Links:
- removed link 15
- removed link 19
- removed link 210
- removed link 211
- removed link 212
- removed link 23
- removed link 24
- removed link 26
- removed link 27
- removed link 28
- link 0: mass 0.20857165140119374 -> 0.1266106424782611; geometry collision cylinder length=0.5641479681169879 radius=0.26727827258799963; visual cylinder length=0.5641479681169879 radius=0.26727827258799963
- link 11: mass 1.9405244574842238 -> 1.0813750656931778; geometry collision cylinder length=0.3991762151685897 radius=0.9286047724461834; visual cylinder length=0.3991762151685897 radius=0.9286047724461834
- link 22: mass 0.151363857123784 -> 0.1719826557781397; geometry collision cylinder length=0.9913247191047079 radius=0.23499543261728517; visual cylinder length=0.9913247191047079 radius=0.23499543261728517
Joints:
- removed joint 15_to_0
- removed joint 19_to_0
- removed joint 210_to_19
- removed joint 211_to_19
- removed joint 212_to_19
- removed joint 22_to_11
- removed joint 23_to_11
- removed joint 24_to_11
- removed joint 26_to_15
- removed joint 27_to_15
- removed joint 28_to_15
- added joint 22_to_0: type revolute, parent 0, child 22, origin xyz=0.05201508349126427 0.8442719017248157 0.520904250296006 rpy=10.082666290617706 1.308169514647243 3.285481549493712, axis 1 0 0, limit lower=3.1415 upper=-3.1415 effort=1 velocity=1
- joint 11_to_0: axis 1 0 0 -> 0 0 1; origin xyz=0.7664424799162463 0.03336009499702208 0.5976603961001847 rpy=1.8690657813970295 0.3060370046931864 4.032123634108947 -> xyz=0.47937751848951704 0.17493281279465944 0.12482231719935388 rpy=0.17934487013463388 5.346351575067694 4.607088505421354
