Commit message: done with eval population without threading

File: test.urdf (robot description, URDF)
Before this commit: robot jiejie, 7 links, 6 joints
Links:
- removed link 23
- removed link 35
- removed link 36
- removed link 42
- added link 120, mass 0.31074178119963686; collision cylinder length=0.3028600532102631 radius=0.57148375797038; visual cylinder length=0.3028600532102631 radius=0.57148375797038
- added link 139, mass 0.31074178119963686; collision cylinder length=0.3028600532102631 radius=0.57148375797038; visual cylinder length=0.3028600532102631 radius=0.57148375797038
- added link 158, mass 0.31074178119963686; collision cylinder length=0.3028600532102631 radius=0.57148375797038; visual cylinder length=0.3028600532102631 radius=0.57148375797038
- added link 214, mass 0.8488582945134865; collision cylinder length=0.49523593097411933 radius=0.7386464053728978; visual cylinder length=0.49523593097411933 radius=0.7386464053728978
- added link 22, mass 0.8488582945134865; collision cylinder length=0.49523593097411933 radius=0.7386464053728978; visual cylinder length=0.49523593097411933 radius=0.7386464053728978
- added link 221, mass 0.8488582945134865; collision cylinder length=0.49523593097411933 radius=0.7386464053728978; visual cylinder length=0.49523593097411933 radius=0.7386464053728978
- added link 227, mass 0.8488582945134865; collision cylinder length=0.49523593097411933 radius=0.7386464053728978; visual cylinder length=0.49523593097411933 radius=0.7386464053728978
- added link 233, mass 0.8488582945134865; collision cylinder length=0.49523593097411933 radius=0.7386464053728978; visual cylinder length=0.49523593097411933 radius=0.7386464053728978
- added link 240, mass 0.8488582945134865; collision cylinder length=0.49523593097411933 radius=0.7386464053728978; visual cylinder length=0.49523593097411933 radius=0.7386464053728978
- added link 246, mass 0.8488582945134865; collision cylinder length=0.49523593097411933 radius=0.7386464053728978; visual cylinder length=0.49523593097411933 radius=0.7386464053728978
- added link 252, mass 0.8488582945134865; collision cylinder length=0.49523593097411933 radius=0.7386464053728978; visual cylinder length=0.49523593097411933 radius=0.7386464053728978
- added link 259, mass 0.8488582945134865; collision cylinder length=0.49523593097411933 radius=0.7386464053728978; visual cylinder length=0.49523593097411933 radius=0.7386464053728978
- added link 265, mass 0.8488582945134865; collision cylinder length=0.49523593097411933 radius=0.7386464053728978; visual cylinder length=0.49523593097411933 radius=0.7386464053728978
- added link 271, mass 0.8488582945134865; collision cylinder length=0.49523593097411933 radius=0.7386464053728978; visual cylinder length=0.49523593097411933 radius=0.7386464053728978
- added link 28, mass 0.8488582945134865; collision cylinder length=0.49523593097411933 radius=0.7386464053728978; visual cylinder length=0.49523593097411933 radius=0.7386464053728978
- added link 310, mass 0.2903371030951946; collision cylinder length=0.2249928859473701 radius=0.6409024622643849; visual cylinder length=0.2249928859473701 radius=0.6409024622643849
- added link 315, mass 0.2903371030951946; collision cylinder length=0.2249928859473701 radius=0.6409024622643849; visual cylinder length=0.2249928859473701 radius=0.6409024622643849
- added link 316, mass 0.2903371030951946; collision cylinder length=0.2249928859473701 radius=0.6409024622643849; visual cylinder length=0.2249928859473701 radius=0.6409024622643849
- added link 322, mass 0.2903371030951946; collision cylinder length=0.2249928859473701 radius=0.6409024622643849; visual cylinder length=0.2249928859473701 radius=0.6409024622643849
- added link 323, mass 0.2903371030951946; collision cylinder length=0.2249928859473701 radius=0.6409024622643849; visual cylinder length=0.2249928859473701 radius=0.6409024622643849
- added link 328, mass 0.2903371030951946; collision cylinder length=0.2249928859473701 radius=0.6409024622643849; visual cylinder length=0.2249928859473701 radius=0.6409024622643849
- added link 329, mass 0.2903371030951946; collision cylinder length=0.2249928859473701 radius=0.6409024622643849; visual cylinder length=0.2249928859473701 radius=0.6409024622643849
- added link 33, mass 0.2903371030951946; collision cylinder length=0.2249928859473701 radius=0.6409024622643849; visual cylinder length=0.2249928859473701 radius=0.6409024622643849
- added link 334, mass 0.2903371030951946; collision cylinder length=0.2249928859473701 radius=0.6409024622643849; visual cylinder length=0.2249928859473701 radius=0.6409024622643849
- added link 335, mass 0.2903371030951946; collision cylinder length=0.2249928859473701 radius=0.6409024622643849; visual cylinder length=0.2249928859473701 radius=0.6409024622643849
- added link 341, mass 0.2903371030951946; collision cylinder length=0.2249928859473701 radius=0.6409024622643849; visual cylinder length=0.2249928859473701 radius=0.6409024622643849
- added link 342, mass 0.2903371030951946; collision cylinder length=0.2249928859473701 radius=0.6409024622643849; visual cylinder length=0.2249928859473701 radius=0.6409024622643849
- added link 347, mass 0.2903371030951946; collision cylinder length=0.2249928859473701 radius=0.6409024622643849; visual cylinder length=0.2249928859473701 radius=0.6409024622643849
- added link 348, mass 0.2903371030951946; collision cylinder length=0.2249928859473701 radius=0.6409024622643849; visual cylinder length=0.2249928859473701 radius=0.6409024622643849
- added link 353, mass 0.2903371030951946; collision cylinder length=0.2249928859473701 radius=0.6409024622643849; visual cylinder length=0.2249928859473701 radius=0.6409024622643849
- added link 354, mass 0.2903371030951946; collision cylinder length=0.2249928859473701 radius=0.6409024622643849; visual cylinder length=0.2249928859473701 radius=0.6409024622643849
- added link 360, mass 0.2903371030951946; collision cylinder length=0.2249928859473701 radius=0.6409024622643849; visual cylinder length=0.2249928859473701 radius=0.6409024622643849
- added link 361, mass 0.2903371030951946; collision cylinder length=0.2249928859473701 radius=0.6409024622643849; visual cylinder length=0.2249928859473701 radius=0.6409024622643849
- added link 366, mass 0.2903371030951946; collision cylinder length=0.2249928859473701 radius=0.6409024622643849; visual cylinder length=0.2249928859473701 radius=0.6409024622643849
- added link 367, mass 0.2903371030951946; collision cylinder length=0.2249928859473701 radius=0.6409024622643849; visual cylinder length=0.2249928859473701 radius=0.6409024622643849
- added link 372, mass 0.2903371030951946; collision cylinder length=0.2249928859473701 radius=0.6409024622643849; visual cylinder length=0.2249928859473701 radius=0.6409024622643849
- added link 373, mass 0.2903371030951946; collision cylinder length=0.2249928859473701 radius=0.6409024622643849; visual cylinder length=0.2249928859473701 radius=0.6409024622643849
- added link 39, mass 0.2903371030951946; collision cylinder length=0.2249928859473701 radius=0.6409024622643849; visual cylinder length=0.2249928859473701 radius=0.6409024622643849
- added link 411, mass 0.13623306899209547; collision cylinder length=0.11916902576509247 radius=0.6032323717084854; visual cylinder length=0.11916902576509247 radius=0.6032323717084854
- added link 412, mass 0.13623306899209547; collision cylinder length=0.11916902576509247 radius=0.6032323717084854; visual cylinder length=0.11916902576509247 radius=0.6032323717084854
- added link 413, mass 0.13623306899209547; collision cylinder length=0.11916902576509247 radius=0.6032323717084854; visual cylinder length=0.11916902576509247 radius=0.6032323717084854
- added link 417, mass 0.13623306899209547; collision cylinder length=0.11916902576509247 radius=0.6032323717084854; visual cylinder length=0.11916902576509247 radius=0.6032323717084854
- added link 418, mass 0.13623306899209547; collision cylinder length=0.11916902576509247 radius=0.6032323717084854; visual cylinder length=0.11916902576509247 radius=0.6032323717084854
- added link 419, mass 0.13623306899209547; collision cylinder length=0.11916902576509247 radius=0.6032323717084854; visual cylinder length=0.11916902576509247 radius=0.6032323717084854
- added link 424, mass 0.13623306899209547; collision cylinder length=0.11916902576509247 radius=0.6032323717084854; visual cylinder length=0.11916902576509247 radius=0.6032323717084854
- added link 425, mass 0.13623306899209547; collision cylinder length=0.11916902576509247 radius=0.6032323717084854; visual cylinder length=0.11916902576509247 radius=0.6032323717084854
- added link 426, mass 0.13623306899209547; collision cylinder length=0.11916902576509247 radius=0.6032323717084854; visual cylinder length=0.11916902576509247 radius=0.6032323717084854
- added link 430, mass 0.13623306899209547; collision cylinder length=0.11916902576509247 radius=0.6032323717084854; visual cylinder length=0.11916902576509247 radius=0.6032323717084854
- added link 431, mass 0.13623306899209547; collision cylinder length=0.11916902576509247 radius=0.6032323717084854; visual cylinder length=0.11916902576509247 radius=0.6032323717084854
- added link 432, mass 0.13623306899209547; collision cylinder length=0.11916902576509247 radius=0.6032323717084854; visual cylinder length=0.11916902576509247 radius=0.6032323717084854
- added link 436, mass 0.13623306899209547; collision cylinder length=0.11916902576509247 radius=0.6032323717084854; visual cylinder length=0.11916902576509247 radius=0.6032323717084854
- added link 437, mass 0.13623306899209547; collision cylinder length=0.11916902576509247 radius=0.6032323717084854; visual cylinder length=0.11916902576509247 radius=0.6032323717084854
- added link 438, mass 0.13623306899209547; collision cylinder length=0.11916902576509247 radius=0.6032323717084854; visual cylinder length=0.11916902576509247 radius=0.6032323717084854
- added link 443, mass 0.13623306899209547; collision cylinder length=0.11916902576509247 radius=0.6032323717084854; visual cylinder length=0.11916902576509247 radius=0.6032323717084854
- added link 444, mass 0.13623306899209547; collision cylinder length=0.11916902576509247 radius=0.6032323717084854; visual cylinder length=0.11916902576509247 radius=0.6032323717084854
- added link 445, mass 0.13623306899209547; collision cylinder length=0.11916902576509247 radius=0.6032323717084854; visual cylinder length=0.11916902576509247 radius=0.6032323717084854
- added link 449, mass 0.13623306899209547; collision cylinder length=0.11916902576509247 radius=0.6032323717084854; visual cylinder length=0.11916902576509247 radius=0.6032323717084854
- added link 45, mass 0.13623306899209547; collision cylinder length=0.11916902576509247 radius=0.6032323717084854; visual cylinder length=0.11916902576509247 radius=0.6032323717084854
- added link 450, mass 0.13623306899209547; collision cylinder length=0.11916902576509247 radius=0.6032323717084854; visual cylinder length=0.11916902576509247 radius=0.6032323717084854
- added link 451, mass 0.13623306899209547; collision cylinder length=0.11916902576509247 radius=0.6032323717084854; visual cylinder length=0.11916902576509247 radius=0.6032323717084854
- added link 455, mass 0.13623306899209547; collision cylinder length=0.11916902576509247 radius=0.6032323717084854; visual cylinder length=0.11916902576509247 radius=0.6032323717084854
- added link 456, mass 0.13623306899209547; collision cylinder length=0.11916902576509247 radius=0.6032323717084854; visual cylinder length=0.11916902576509247 radius=0.6032323717084854
- added link 457, mass 0.13623306899209547; collision cylinder length=0.11916902576509247 radius=0.6032323717084854; visual cylinder length=0.11916902576509247 radius=0.6032323717084854
- added link 46, mass 0.13623306899209547; collision cylinder length=0.11916902576509247 radius=0.6032323717084854; visual cylinder length=0.11916902576509247 radius=0.6032323717084854
- added link 462, mass 0.13623306899209547; collision cylinder length=0.11916902576509247 radius=0.6032323717084854; visual cylinder length=0.11916902576509247 radius=0.6032323717084854
- added link 463, mass 0.13623306899209547; collision cylinder length=0.11916902576509247 radius=0.6032323717084854; visual cylinder length=0.11916902576509247 radius=0.6032323717084854
- added link 464, mass 0.13623306899209547; collision cylinder length=0.11916902576509247 radius=0.6032323717084854; visual cylinder length=0.11916902576509247 radius=0.6032323717084854
- added link 468, mass 0.13623306899209547; collision cylinder length=0.11916902576509247 radius=0.6032323717084854; visual cylinder length=0.11916902576509247 radius=0.6032323717084854
- added link 469, mass 0.13623306899209547; collision cylinder length=0.11916902576509247 radius=0.6032323717084854; visual cylinder length=0.11916902576509247 radius=0.6032323717084854
- added link 47, mass 0.13623306899209547; collision cylinder length=0.11916902576509247 radius=0.6032323717084854; visual cylinder length=0.11916902576509247 radius=0.6032323717084854
- added link 470, mass 0.13623306899209547; collision cylinder length=0.11916902576509247 radius=0.6032323717084854; visual cylinder length=0.11916902576509247 radius=0.6032323717084854
- added link 474, mass 0.13623306899209547; collision cylinder length=0.11916902576509247 radius=0.6032323717084854; visual cylinder length=0.11916902576509247 radius=0.6032323717084854
- added link 475, mass 0.13623306899209547; collision cylinder length=0.11916902576509247 radius=0.6032323717084854; visual cylinder length=0.11916902576509247 radius=0.6032323717084854
- added link 476, mass 0.13623306899209547; collision cylinder length=0.11916902576509247 radius=0.6032323717084854; visual cylinder length=0.11916902576509247 radius=0.6032323717084854
- link 0: mass 1.4496508885561628 -> 1.016272175300422; geometry collision cylinder length=0.32773470592924947 radius=0.9935022710170807; visual cylinder length=0.32773470592924947 radius=0.9935022710170807
- link 11: mass 3.0396257637464026 -> 0.31074178119963686; geometry collision cylinder length=0.3028600532102631 radius=0.57148375797038; visual cylinder length=0.3028600532102631 radius=0.57148375797038
- link 34: mass 2.567585560992488 -> 0.2903371030951946; geometry collision cylinder length=0.2249928859473701 radius=0.6409024622643849; visual cylinder length=0.2249928859473701 radius=0.6409024622643849
Joints:
- removed joint 23_to_0
- removed joint 34_to_0
- removed joint 35_to_0
- removed joint 36_to_0
- removed joint 42_to_11
- added joint 120_to_0: type revolute, parent 0, child 120, origin xyz=0.5519166036276144 0.02006754526396426 0.5872844150574494 rpy=18.223957745966974 0.6342158404441013 4.866742757937005, axis 0 1 0, limit lower=3.1415 upper=-3.1415 effort=1 velocity=1
- added joint 139_to_0: type revolute, parent 0, child 139, origin xyz=0.5519166036276144 0.02006754526396426 0.5872844150574494 rpy=24.298610327955966 0.6342158404441013 4.866742757937005, axis 0 1 0, limit lower=3.1415 upper=-3.1415 effort=1 velocity=1
- added joint 158_to_0: type revolute, parent 0, child 158, origin xyz=0.5519166036276144 0.02006754526396426 0.5872844150574494 rpy=30.37326290994496 0.6342158404441013 4.866742757937005, axis 0 1 0, limit lower=3.1415 upper=-3.1415 effort=1 velocity=1
- added joint 214_to_11: type revolute, parent 11, child 214, origin xyz=0.15971455959588698 0.7748798714524615 0.6515819450043923 rpy=1.7590457093358354 4.467210131069551 5.917120936824633, axis 1 0 0, limit lower=3.1415 upper=-3.1415 effort=1 velocity=1
- added joint 221_to_120: type revolute, parent 120, child 221, origin xyz=0.15971455959588698 0.7748798714524615 0.6515819450043923 rpy=0.8795228546679177 4.467210131069551 5.917120936824633, axis 1 0 0, limit lower=3.1415 upper=-3.1415 effort=1 velocity=1
- added joint 227_to_120: type revolute, parent 120, child 227, origin xyz=0.15971455959588698 0.7748798714524615 0.6515819450043923 rpy=1.3192842820018766 4.467210131069551 5.917120936824633, axis 1 0 0, limit lower=3.1415 upper=-3.1415 effort=1 velocity=1
- added joint 22_to_11: type revolute, parent 11, child 22, origin xyz=0.15971455959588698 0.7748798714524615 0.6515819450043923 rpy=0.8795228546679177 4.467210131069551 5.917120936824633, axis 1 0 0, limit lower=3.1415 upper=-3.1415 effort=1 velocity=1
- added joint 233_to_120: type revolute, parent 120, child 233, origin xyz=0.15971455959588698 0.7748798714524615 0.6515819450043923 rpy=1.7590457093358354 4.467210131069551 5.917120936824633, axis 1 0 0, limit lower=3.1415 upper=-3.1415 effort=1 velocity=1
- added joint 240_to_139: type revolute, parent 139, child 240, origin xyz=0.15971455959588698 0.7748798714524615 0.6515819450043923 rpy=0.8795228546679177 4.467210131069551 5.917120936824633, axis 1 0 0, limit lower=3.1415 upper=-3.1415 effort=1 velocity=1
- added joint 246_to_139: type revolute, parent 139, child 246, origin xyz=0.15971455959588698 0.7748798714524615 0.6515819450043923 rpy=1.3192842820018766 4.467210131069551 5.917120936824633, axis 1 0 0, limit lower=3.1415 upper=-3.1415 effort=1 velocity=1
- added joint 252_to_139: type revolute, parent 139, child 252, origin xyz=0.15971455959588698 0.7748798714524615 0.6515819450043923 rpy=1.7590457093358354 4.467210131069551 5.917120936824633, axis 1 0 0, limit lower=3.1415 upper=-3.1415 effort=1 velocity=1
- added joint 259_to_158: type revolute, parent 158, child 259, origin xyz=0.15971455959588698 0.7748798714524615 0.6515819450043923 rpy=0.8795228546679177 4.467210131069551 5.917120936824633, axis 1 0 0, limit lower=3.1415 upper=-3.1415 effort=1 velocity=1
- added joint 265_to_158: type revolute, parent 158, child 265, origin xyz=0.15971455959588698 0.7748798714524615 0.6515819450043923 rpy=1.3192842820018766 4.467210131069551 5.917120936824633, axis 1 0 0, limit lower=3.1415 upper=-3.1415 effort=1 velocity=1
- added joint 271_to_158: type revolute, parent 158, child 271, origin xyz=0.15971455959588698 0.7748798714524615 0.6515819450043923 rpy=1.7590457093358354 4.467210131069551 5.917120936824633, axis 1 0 0, limit lower=3.1415 upper=-3.1415 effort=1 velocity=1
- added joint 28_to_11: type revolute, parent 11, child 28, origin xyz=0.15971455959588698 0.7748798714524615 0.6515819450043923 rpy=1.3192842820018766 4.467210131069551 5.917120936824633, axis 1 0 0, limit lower=3.1415 upper=-3.1415 effort=1 velocity=1
- added joint 310_to_28: type revolute, parent 28, child 310, origin xyz=0.5523001038389661 0.04334783898074657 0.20593450716308614 rpy=15.549335322884257 3.6989156431602352 0.17073447837032898, axis 1 0 0, limit lower=3.1415 upper=-3.1415 effort=1 velocity=1
- added joint 315_to_214: type revolute, parent 214, child 315, origin xyz=0.5523001038389661 0.04334783898074657 0.20593450716308614 rpy=10.366223548589504 3.6989156431602352 0.17073447837032898, axis 1 0 0, limit lower=3.1415 upper=-3.1415 effort=1 velocity=1
- added joint 316_to_214: type revolute, parent 214, child 316, origin xyz=0.5523001038389661 0.04334783898074657 0.20593450716308614 rpy=15.549335322884257 3.6989156431602352 0.17073447837032898, axis 1 0 0, limit lower=3.1415 upper=-3.1415 effort=1 velocity=1
- added joint 322_to_221: type revolute, parent 221, child 322, origin xyz=0.5523001038389661 0.04334783898074657 0.20593450716308614 rpy=10.366223548589504 3.6989156431602352 0.17073447837032898, axis 1 0 0, limit lower=3.1415 upper=-3.1415 effort=1 velocity=1
- added joint 323_to_221: type revolute, parent 221, child 323, origin xyz=0.5523001038389661 0.04334783898074657 0.20593450716308614 rpy=15.549335322884257 3.6989156431602352 0.17073447837032898, axis 1 0 0, limit lower=3.1415 upper=-3.1415 effort=1 velocity=1
- added joint 328_to_227: type revolute, parent 227, child 328, origin xyz=0.5523001038389661 0.04334783898074657 0.20593450716308614 rpy=10.366223548589504 3.6989156431602352 0.17073447837032898, axis 1 0 0, limit lower=3.1415 upper=-3.1415 effort=1 velocity=1
- added joint 329_to_227: type revolute, parent 227, child 329, origin xyz=0.5523001038389661 0.04334783898074657 0.20593450716308614 rpy=15.549335322884257 3.6989156431602352 0.17073447837032898, axis 1 0 0, limit lower=3.1415 upper=-3.1415 effort=1 velocity=1
- added joint 334_to_233: type revolute, parent 233, child 334, origin xyz=0.5523001038389661 0.04334783898074657 0.20593450716308614 rpy=10.366223548589504 3.6989156431602352 0.17073447837032898, axis 1 0 0, limit lower=3.1415 upper=-3.1415 effort=1 velocity=1
- added joint 335_to_233: type revolute, parent 233, child 335, origin xyz=0.5523001038389661 0.04334783898074657 0.20593450716308614 rpy=15.549335322884257 3.6989156431602352 0.17073447837032898, axis 1 0 0, limit lower=3.1415 upper=-3.1415 effort=1 velocity=1
- added joint 33_to_22: type revolute, parent 22, child 33, origin xyz=0.5523001038389661 0.04334783898074657 0.20593450716308614 rpy=10.366223548589504 3.6989156431602352 0.17073447837032898, axis 1 0 0, limit lower=3.1415 upper=-3.1415 effort=1 velocity=1
- added joint 341_to_240: type revolute, parent 240, child 341, origin xyz=0.5523001038389661 0.04334783898074657 0.20593450716308614 rpy=10.366223548589504 3.6989156431602352 0.17073447837032898, axis 1 0 0, limit lower=3.1415 upper=-3.1415 effort=1 velocity=1
- added joint 342_to_240: type revolute, parent 240, child 342, origin xyz=0.5523001038389661 0.04334783898074657 0.20593450716308614 rpy=15.549335322884257 3.6989156431602352 0.17073447837032898, axis 1 0 0, limit lower=3.1415 upper=-3.1415 effort=1 velocity=1
- added joint 347_to_246: type revolute, parent 246, child 347, origin xyz=0.5523001038389661 0.04334783898074657 0.20593450716308614 rpy=10.366223548589504 3.6989156431602352 0.17073447837032898, axis 1 0 0, limit lower=3.1415 upper=-3.1415 effort=1 velocity=1
- added joint 348_to_246: type revolute, parent 246, child 348, origin xyz=0.5523001038389661 0.04334783898074657 0.20593450716308614 rpy=15.549335322884257 3.6989156431602352 0.17073447837032898, axis 1 0 0, limit lower=3.1415 upper=-3.1415 effort=1 velocity=1
- added joint 34_to_22: type revolute, parent 22, child 34, origin xyz=0.5523001038389661 0.04334783898074657 0.20593450716308614 rpy=15.549335322884257 3.6989156431602352 0.17073447837032898, axis 1 0 0, limit lower=3.1415 upper=-3.1415 effort=1 velocity=1
- added joint 353_to_252: type revolute, parent 252, child 353, origin xyz=0.5523001038389661 0.04334783898074657 0.20593450716308614 rpy=10.366223548589504 3.6989156431602352 0.17073447837032898, axis 1 0 0, limit lower=3.1415 upper=-3.1415 effort=1 velocity=1
- added joint 354_to_252: type revolute, parent 252, child 354, origin xyz=0.5523001038389661 0.04334783898074657 0.20593450716308614 rpy=15.549335322884257 3.6989156431602352 0.17073447837032898, axis 1 0 0, limit lower=3.1415 upper=-3.1415 effort=1 velocity=1
- added joint 360_to_259: type revolute, parent 259, child 360, origin xyz=0.5523001038389661 0.04334783898074657 0.20593450716308614 rpy=10.366223548589504 3.6989156431602352 0.17073447837032898, axis 1 0 0, limit lower=3.1415 upper=-3.1415 effort=1 velocity=1
- added joint 361_to_259: type revolute, parent 259, child 361, origin xyz=0.5523001038389661 0.04334783898074657 0.20593450716308614 rpy=15.549335322884257 3.6989156431602352 0.17073447837032898, axis 1 0 0, limit lower=3.1415 upper=-3.1415 effort=1 velocity=1
- added joint 366_to_265: type revolute, parent 265, child 366, origin xyz=0.5523001038389661 0.04334783898074657 0.20593450716308614 rpy=10.366223548589504 3.6989156431602352 0.17073447837032898, axis 1 0 0, limit lower=3.1415 upper=-3.1415 effort=1 velocity=1
- added joint 367_to_265: type revolute, parent 265, child 367, origin xyz=0.5523001038389661 0.04334783898074657 0.20593450716308614 rpy=15.549335322884257 3.6989156431602352 0.17073447837032898, axis 1 0 0, limit lower=3.1415 upper=-3.1415 effort=1 velocity=1
- added joint 372_to_271: type revolute, parent 271, child 372, origin xyz=0.5523001038389661 0.04334783898074657 0.20593450716308614 rpy=10.366223548589504 3.6989156431602352 0.17073447837032898, axis 1 0 0, limit lower=3.1415 upper=-3.1415 effort=1 velocity=1
- added joint 373_to_271: type revolute, parent 271, child 373, origin xyz=0.5523001038389661 0.04334783898074657 0.20593450716308614 rpy=15.549335322884257 3.6989156431602352 0.17073447837032898, axis 1 0 0, limit lower=3.1415 upper=-3.1415 effort=1 velocity=1
- added joint 39_to_28: type revolute, parent 28, child 39, origin xyz=0.5523001038389661 0.04334783898074657 0.20593450716308614 rpy=10.366223548589504 3.6989156431602352 0.17073447837032898, axis 1 0 0, limit lower=3.1415 upper=-3.1415 effort=1 velocity=1
- added joint 411_to_28: type revolute, parent 28, child 411, origin xyz=0.31582333589701006 0.4438536130406737 0.38918718471101754 rpy=22.175685651460288 1.4151809419677086 5.406214837045536, axis 0 1 0, limit lower=3.1415 upper=-3.1415 effort=1 velocity=1
- added joint 412_to_28: type revolute, parent 28, child 412, origin xyz=0.31582333589701006 0.4438536130406737 0.38918718471101754 rpy=27.71960706432536 1.4151809419677086 5.406214837045536, axis 0 1 0, limit lower=3.1415 upper=-3.1415 effort=1 velocity=1
- added joint 413_to_28: type revolute, parent 28, child 413, origin xyz=0.31582333589701006 0.4438536130406737 0.38918718471101754 rpy=33.263528477190434 1.4151809419677086 5.406214837045536, axis 0 1 0, limit lower=3.1415 upper=-3.1415 effort=1 velocity=1
- added joint 417_to_214: type revolute, parent 214, child 417, origin xyz=0.31582333589701006 0.4438536130406737 0.38918718471101754 rpy=22.175685651460288 1.4151809419677086 5.406214837045536, axis 0 1 0, limit lower=3.1415 upper=-3.1415 effort=1 velocity=1
- added joint 418_to_214: type revolute, parent 214, child 418, origin xyz=0.31582333589701006 0.4438536130406737 0.38918718471101754 rpy=27.71960706432536 1.4151809419677086 5.406214837045536, axis 0 1 0, limit lower=3.1415 upper=-3.1415 effort=1 velocity=1
- added joint 419_to_214: type revolute, parent 214, child 419, origin xyz=0.31582333589701006 0.4438536130406737 0.38918718471101754 rpy=33.263528477190434 1.4151809419677086 5.406214837045536, axis 0 1 0, limit lower=3.1415 upper=-3.1415 effort=1 velocity=1
- added joint 424_to_221: type revolute, parent 221, child 424, origin xyz=0.31582333589701006 0.4438536130406737 0.38918718471101754 rpy=22.175685651460288 1.4151809419677086 5.406214837045536, axis 0 1 0, limit lower=3.1415 upper=-3.1415 effort=1 velocity=1
- added joint 425_to_221: type revolute, parent 221, child 425, origin xyz=0.31582333589701006 0.4438536130406737 0.38918718471101754 rpy=27.71960706432536 1.4151809419677086 5.406214837045536, axis 0 1 0, limit lower=3.1415 upper=-3.1415 effort=1 velocity=1
- added joint 426_to_221: type revolute, parent 221, child 426, origin xyz=0.31582333589701006 0.4438536130406737 0.38918718471101754 rpy=33.263528477190434 1.4151809419677086 5.406214837045536, axis 0 1 0, limit lower=3.1415 upper=-3.1415 effort=1 velocity=1
- added joint 430_to_227: type revolute, parent 227, child 430, origin xyz=0.31582333589701006 0.4438536130406737 0.38918718471101754 rpy=22.175685651460288 1.4151809419677086 5.406214837045536, axis 0 1 0, limit lower=3.1415 upper=-3.1415 effort=1 velocity=1
- added joint 431_to_227: type revolute, parent 227, child 431, origin xyz=0.31582333589701006 0.4438536130406737 0.38918718471101754 rpy=27.71960706432536 1.4151809419677086 5.406214837045536, axis 0 1 0, limit lower=3.1415 upper=-3.1415 effort=1 velocity=1
- added joint 432_to_227: type revolute, parent 227, child 432, origin xyz=0.31582333589701006 0.4438536130406737 0.38918718471101754 rpy=33.263528477190434 1.4151809419677086 5.406214837045536, axis 0 1 0, limit lower=3.1415 upper=-3.1415 effort=1 velocity=1
- added joint 436_to_233: type revolute, parent 233, child 436, origin xyz=0.31582333589701006 0.4438536130406737 0.38918718471101754 rpy=22.175685651460288 1.4151809419677086 5.406214837045536, axis 0 1 0, limit lower=3.1415 upper=-3.1415 effort=1 velocity=1
- added joint 437_to_233: type revolute, parent 233, child 437, origin xyz=0.31582333589701006 0.4438536130406737 0.38918718471101754 rpy=27.71960706432536 1.4151809419677086 5.406214837045536, axis 0 1 0, limit lower=3.1415 upper=-3.1415 effort=1 velocity=1
- added joint 438_to_233: type revolute, parent 233, child 438, origin xyz=0.31582333589701006 0.4438536130406737 0.38918718471101754 rpy=33.263528477190434 1.4151809419677086 5.406214837045536, axis 0 1 0, limit lower=3.1415 upper=-3.1415 effort=1 velocity=1
- added joint 443_to_240: type revolute, parent 240, child 443, origin xyz=0.31582333589701006 0.4438536130406737 0.38918718471101754 rpy=22.175685651460288 1.4151809419677086 5.406214837045536, axis 0 1 0, limit lower=3.1415 upper=-3.1415 effort=1 velocity=1
- added joint 444_to_240: type revolute, parent 240, child 444, origin xyz=0.31582333589701006 0.4438536130406737 0.38918718471101754 rpy=27.71960706432536 1.4151809419677086 5.406214837045536, axis 0 1 0, limit lower=3.1415 upper=-3.1415 effort=1 velocity=1
- added joint 445_to_240: type revolute, parent 240, child 445, origin xyz=0.31582333589701006 0.4438536130406737 0.38918718471101754 rpy=33.263528477190434 1.4151809419677086 5.406214837045536, axis 0 1 0, limit lower=3.1415 upper=-3.1415 effort=1 velocity=1
- added joint 449_to_246: type revolute, parent 246, child 449, origin xyz=0.31582333589701006 0.4438536130406737 0.38918718471101754 rpy=22.175685651460288 1.4151809419677086 5.406214837045536, axis 0 1 0, limit lower=3.1415 upper=-3.1415 effort=1 velocity=1
- added joint 450_to_246: type revolute, parent 246, child 450, origin xyz=0.31582333589701006 0.4438536130406737 0.38918718471101754 rpy=27.71960706432536 1.4151809419677086 5.406214837045536, axis 0 1 0, limit lower=3.1415 upper=-3.1415 effort=1 velocity=1
- added joint 451_to_246: type revolute, parent 246, child 451, origin xyz=0.31582333589701006 0.4438536130406737 0.38918718471101754 rpy=33.263528477190434 1.4151809419677086 5.406214837045536, axis 0 1 0, limit lower=3.1415 upper=-3.1415 effort=1 velocity=1
- added joint 455_to_252: type revolute, parent 252, child 455, origin xyz=0.31582333589701006 0.4438536130406737 0.38918718471101754 rpy=22.175685651460288 1.4151809419677086 5.406214837045536, axis 0 1 0, limit lower=3.1415 upper=-3.1415 effort=1 velocity=1
- added joint 456_to_252: type revolute, parent 252, child 456, origin xyz=0.31582333589701006 0.4438536130406737 0.38918718471101754 rpy=27.71960706432536 1.4151809419677086 5.406214837045536, axis 0 1 0, limit lower=3.1415 upper=-3.1415 effort=1 velocity=1
- added joint 457_to_252: type revolute, parent 252, child 457, origin xyz=0.31582333589701006 0.4438536130406737 0.38918718471101754 rpy=33.263528477190434 1.4151809419677086 5.406214837045536, axis 0 1 0, limit lower=3.1415 upper=-3.1415 effort=1 velocity=1
- added joint 45_to_22: type revolute, parent 22, child 45, origin xyz=0.31582333589701006 0.4438536130406737 0.38918718471101754 rpy=22.175685651460288 1.4151809419677086 5.406214837045536, axis 0 1 0, limit lower=3.1415 upper=-3.1415 effort=1 velocity=1
- added joint 462_to_259: type revolute, parent 259, child 462, origin xyz=0.31582333589701006 0.4438536130406737 0.38918718471101754 rpy=22.175685651460288 1.4151809419677086 5.406214837045536, axis 0 1 0, limit lower=3.1415 upper=-3.1415 effort=1 velocity=1
- added joint 463_to_259: type revolute, parent 259, child 463, origin xyz=0.31582333589701006 0.4438536130406737 0.38918718471101754 rpy=27.71960706432536 1.4151809419677086 5.406214837045536, axis 0 1 0, limit lower=3.1415 upper=-3.1415 effort=1 velocity=1
- added joint 464_to_259: type revolute, parent 259, child 464, origin xyz=0.31582333589701006 0.4438536130406737 0.38918718471101754 rpy=33.263528477190434 1.4151809419677086 5.406214837045536, axis 0 1 0, limit lower=3.1415 upper=-3.1415 effort=1 velocity=1
- added joint 468_to_265: type revolute, parent 265, child 468, origin xyz=0.31582333589701006 0.4438536130406737 0.38918718471101754 rpy=22.175685651460288 1.4151809419677086 5.406214837045536, axis 0 1 0, limit lower=3.1415 upper=-3.1415 effort=1 velocity=1
- added joint 469_to_265: type revolute, parent 265, child 469, origin xyz=0.31582333589701006 0.4438536130406737 0.38918718471101754 rpy=27.71960706432536 1.4151809419677086 5.406214837045536, axis 0 1 0, limit lower=3.1415 upper=-3.1415 effort=1 velocity=1
- added joint 46_to_22: type revolute, parent 22, child 46, origin xyz=0.31582333589701006 0.4438536130406737 0.38918718471101754 rpy=27.71960706432536 1.4151809419677086 5.406214837045536, axis 0 1 0, limit lower=3.1415 upper=-3.1415 effort=1 velocity=1
- added joint 470_to_265: type revolute, parent 265, child 470, origin xyz=0.31582333589701006 0.4438536130406737 0.38918718471101754 rpy=33.263528477190434 1.4151809419677086 5.406214837045536, axis 0 1 0, limit lower=3.1415 upper=-3.1415 effort=1 velocity=1
- added joint 474_to_271: type revolute, parent 271, child 474, origin xyz=0.31582333589701006 0.4438536130406737 0.38918718471101754 rpy=22.175685651460288 1.4151809419677086 5.406214837045536, axis 0 1 0, limit lower=3.1415 upper=-3.1415 effort=1 velocity=1
- added joint 475_to_271: type revolute, parent 271, child 475, origin xyz=0.31582333589701006 0.4438536130406737 0.38918718471101754 rpy=27.71960706432536 1.4151809419677086 5.406214837045536, axis 0 1 0, limit lower=3.1415 upper=-3.1415 effort=1 velocity=1
- added joint 476_to_271: type revolute, parent 271, child 476, origin xyz=0.31582333589701006 0.4438536130406737 0.38918718471101754 rpy=33.263528477190434 1.4151809419677086 5.406214837045536, axis 0 1 0, limit lower=3.1415 upper=-3.1415 effort=1 velocity=1
- added joint 47_to_22: type revolute, parent 22, child 47, origin xyz=0.31582333589701006 0.4438536130406737 0.38918718471101754 rpy=33.263528477190434 1.4151809419677086 5.406214837045536, axis 0 1 0, limit lower=3.1415 upper=-3.1415 effort=1 velocity=1
- joint 11_to_0: axis 1 0 0 -> 0 1 0; origin xyz=0.8754732290348459 0.2466628855747902 0.5930333966907028 rpy=11.199576226930786 0.23881372681574062 2.5789398753313333 -> xyz=0.5519166036276144 0.02006754526396426 0.5872844150574494 rpy=12.149305163977983 0.6342158404441013 4.866742757937005
