Commit message: implement the testGA function run the genetic algo

File: temp0.urdf (robot description, URDF)
Before this commit: robot jiejie, 6 links, 5 joints
Links:
- removed link 11
- removed link 12
- removed link 13
- removed link 14
- removed link 25
- link 0: mass 1.3956583113167815 -> 0.028254089561562383; geometry collision cylinder length=0.4291582629693992 radius=0.14476280278576104; visual cylinder length=0.4291582629693992 radius=0.14476280278576104
Joints:
- removed joint 11_to_0
- removed joint 12_to_0
- removed joint 13_to_0
- removed joint 14_to_0
- removed joint 25_to_0

Commit message: implemented elitism

File: temp0.urdf (robot description, URDF)
Before this commit: robot jiejie, 1 links, 0 joints
Links:
- added link 11, mass 0.4115691495401723; collision cylinder length=0.1696582101718408 radius=0.8787372361020335; visual cylinder length=0.1696582101718408 radius=0.8787372361020335
- added link 12, mass 0.4115691495401723; collision cylinder length=0.1696582101718408 radius=0.8787372361020335; visual cylinder length=0.1696582101718408 radius=0.8787372361020335
- link 0: mass 0.028254089561562383 -> 0.018770070376035494; geometry collision cylinder length=0.7486991672668879 radius=0.08933144088981038; visual cylinder length=0.7486991672668879 radius=0.08933144088981038
Joints:
- added joint 11_to_0: type revolute, parent 0, child 11, origin xyz=0.17529991906219577 0.30662185138733866 0.38413639560868507 rpy=11.22658176918001 6.008466973836024 1.344418676329795, axis 0 1 0, limit lower=3.1415 upper=-3.1415 effort=1 velocity=1
- added joint 12_to_0: type revolute, parent 0, child 12, origin xyz=0.17529991906219577 0.30662185138733866 0.38413639560868507 rpy=16.839872653770016 6.008466973836024 1.344418676329795, axis 0 1 0, limit lower=3.1415 upper=-3.1415 effort=1 velocity=1

Commit message: additional file for elitism

File: temp0.urdf (robot description, URDF)
Before this commit: robot jiejie, 3 links, 2 joints
Links:
- removed link 12
- link 0: mass 0.018770070376035494 -> 0.08408816224433927; geometry collision cylinder length=0.18298952852664763 radius=0.38245414760072993; visual cylinder length=0.18298952852664763 radius=0.38245414760072993
- link 11: mass 0.4115691495401723 -> 0.08408816224433927; geometry collision cylinder length=0.18298952852664763 radius=0.38245414760072993; visual cylinder length=0.18298952852664763 radius=0.38245414760072993
Joints:
- removed joint 12_to_0
- joint 11_to_0: origin xyz=0.17529991906219577 0.30662185138733866 0.38413639560868507 rpy=11.22658176918001 6.008466973836024 1.344418676329795 -> xyz=0.2625773472446864 0.9324460415970991 0.8509031450824631 rpy=7.267494167952415 1.7669457045395414 2.512242387429224

Commit message: included saving to and reading from csv

File: temp0.urdf (robot description, URDF)
Before this commit: robot jiejie, 2 links, 1 joints
Links:
- removed link 11
- link 0: mass 0.08408816224433927 -> 1.6742212661303668; geometry collision cylinder length=0.559519380339918 radius=0.975941809622658; visual cylinder length=0.559519380339918 radius=0.975941809622658
Joints:
- removed joint 11_to_0

File: test.urdf (robot description, URDF)
Before this commit: robot jiejie, 77 links, 76 joints
Links:
- removed link 120
- removed link 139
- removed link 158
- removed link 214
- removed link 221
- removed link 227
- removed link 233
- removed link 240
- removed link 246
- removed link 252
- removed link 259
- removed link 265
- removed link 271
- removed link 28
- removed link 310
- removed link 315
- removed link 316
- removed link 322
- removed link 323
- removed link 328
- removed link 329
- removed link 334
- removed link 335
- removed link 341
- removed link 342
- removed link 347
- removed link 348
- removed link 353
- removed link 354
- removed link 360
- removed link 361
- removed link 366
- removed link 367
- removed link 372
- removed link 373
- removed link 39
- removed link 411
- removed link 412
- removed link 413
- removed link 417
- removed link 418
- removed link 419
- removed link 424
- removed link 425
- removed link 426
- removed link 430
- removed link 431
- removed link 432
- removed link 436
- removed link 437
- removed link 438
- removed link 443
- removed link 444
- removed link 445
- removed link 449
- removed link 45
- removed link 450
- removed link 451
- removed link 455
- removed link 456
- removed link 457
- removed link 46
- removed link 462
- removed link 463
- removed link 464
- removed link 468
- removed link 469
- removed link 47
- removed link 470
- removed link 474
- removed link 475
- removed link 476
- added link 35, mass 0.1505471416332198; collision cylinder length=0.24662457314719044 radius=0.4408015850001499; visual cylinder length=0.24662457314719044 radius=0.4408015850001499
- added link 36, mass 0.1505471416332198; collision cylinder length=0.24662457314719044 radius=0.4408015850001499; visual cylinder length=0.24662457314719044 radius=0.4408015850001499
- link 0: mass 1.016272175300422 -> 0.003727133234245166; geometry collision cylinder length=0.26594837793743453 radius=0.06679037004577948; visual cylinder length=0.26594837793743453 radius=0.06679037004577948
- link 11: mass 0.31074178119963686 -> 0.2204409066793055; geometry collision cylinder length=0.6064811733117313 radius=0.34014375051735013; visual cylinder length=0.6064811733117313 radius=0.34014375051735013
- link 22: mass 0.8488582945134865 -> 0.36918444014117024; geometry collision cylinder length=0.6538732777368035 radius=0.4239356736584071; visual cylinder length=0.6538732777368035 radius=0.4239356736584071
- link 33: mass 0.2903371030951946 -> 0.1505471416332198; geometry collision cylinder length=0.24662457314719044 radius=0.4408015850001499; visual cylinder length=0.24662457314719044 radius=0.4408015850001499
- link 34: mass 0.2903371030951946 -> 0.1505471416332198; geometry collision cylinder length=0.24662457314719044 radius=0.4408015850001499; visual cylinder length=0.24662457314719044 radius=0.4408015850001499
Joints:
- removed joint 120_to_0
- removed joint 139_to_0
- removed joint 158_to_0
- removed joint 214_to_11
- removed joint 221_to_120
- removed joint 227_to_120
- removed joint 233_to_120
- removed joint 240_to_139
- removed joint 246_to_139
- removed joint 252_to_139
- removed joint 259_to_158
- removed joint 265_to_158
- removed joint 271_to_158
- removed joint 28_to_11
- removed joint 310_to_28
- removed joint 315_to_214
- removed joint 316_to_214
- removed joint 322_to_221
- removed joint 323_to_221
- removed joint 328_to_227
- removed joint 329_to_227
- removed joint 334_to_233
- removed joint 335_to_233
- removed joint 341_to_240
- removed joint 342_to_240
- removed joint 347_to_246
- removed joint 348_to_246
- removed joint 353_to_252
- removed joint 354_to_252
- removed joint 360_to_259
- removed joint 361_to_259
- removed joint 366_to_265
- removed joint 367_to_265
- removed joint 372_to_271
- removed joint 373_to_271
- removed joint 39_to_28
- removed joint 411_to_28
- removed joint 412_to_28
- removed joint 413_to_28
- removed joint 417_to_214
- removed joint 418_to_214
- removed joint 419_to_214
- removed joint 424_to_221
- removed joint 425_to_221
- removed joint 426_to_221
- removed joint 430_to_227
- removed joint 431_to_227
- removed joint 432_to_227
- removed joint 436_to_233
- removed joint 437_to_233
- removed joint 438_to_233
- removed joint 443_to_240
- removed joint 444_to_240
- removed joint 445_to_240
- removed joint 449_to_246
- removed joint 450_to_246
- removed joint 451_to_246
- removed joint 455_to_252
- removed joint 456_to_252
- removed joint 457_to_252
- removed joint 45_to_22
- removed joint 462_to_259
- removed joint 463_to_259
- removed joint 464_to_259
- removed joint 468_to_265
- removed joint 469_to_265
- removed joint 46_to_22
- removed joint 470_to_265
- removed joint 474_to_271
- removed joint 475_to_271
- removed joint 476_to_271
- removed joint 47_to_22
- added joint 35_to_22: type revolute, parent 22, child 35, origin xyz=0.006606340913959841 0.6350182448530621 0.6684790263199062 rpy=12.956592715289158 5.962438929171924 1.5932826144920462, axis 0 1 0, limit lower=3.1415 upper=-3.1415 effort=1 velocity=1
- added joint 36_to_22: type revolute, parent 22, child 36, origin xyz=0.006606340913959841 0.6350182448530621 0.6684790263199062 rpy=16.19574089411145 5.962438929171924 1.5932826144920462, axis 0 1 0, limit lower=3.1415 upper=-3.1415 effort=1 velocity=1
- joint 11_to_0: origin xyz=0.5519166036276144 0.02006754526396426 0.5872844150574494 rpy=12.149305163977983 0.6342158404441013 4.866742757937005 -> xyz=0.5216053173025764 0.6812402403889872 0.7760730921014531 rpy=12.505587441861806 1.9341680253580646 6.2055074284458485
- joint 22_to_11: axis 1 0 0 -> 0 1 0; origin xyz=0.15971455959588698 0.7748798714524615 0.6515819450043923 rpy=0.8795228546679177 4.467210131069551 5.917120936824633 -> xyz=0.3691766231868422 0.5615959505358867 0.1648382158986328 rpy=11.763272034258987 4.835813621793594 4.068722860539795
- joint 33_to_22: axis 1 0 0 -> 0 1 0; origin xyz=0.5523001038389661 0.04334783898074657 0.20593450716308614 rpy=10.366223548589504 3.6989156431602352 0.17073447837032898 -> xyz=0.006606340913959841 0.6350182448530621 0.6684790263199062 rpy=6.478296357644579 5.962438929171924 1.5932826144920462
- joint 34_to_22: axis 1 0 0 -> 0 1 0; origin xyz=0.5523001038389661 0.04334783898074657 0.20593450716308614 rpy=15.549335322884257 3.6989156431602352 0.17073447837032898 -> xyz=0.006606340913959841 0.6350182448530621 0.6684790263199062 rpy=9.717444536466868 5.962438929171924 1.5932826144920462

Commit message: tested on test_ga.py file saved as csv

File: temp0.urdf (robot description, URDF)
Before this commit: robot jiejie, 1 links, 0 joints
Links:
- added link 11, mass 0.12615174120664693; collision cylinder length=0.6621201894926178 radius=0.246265328934829; visual cylinder length=0.6621201894926178 radius=0.246265328934829
- added link 111, mass 0.12615174120664693; collision cylinder length=0.6621201894926178 radius=0.246265328934829; visual cylinder length=0.6621201894926178 radius=0.246265328934829
- added link 16, mass 0.12615174120664693; collision cylinder length=0.6621201894926178 radius=0.246265328934829; visual cylinder length=0.6621201894926178 radius=0.246265328934829
- added link 210, mass 2.3159025717669146; collision cylinder length=0.7373221410868707 radius=0.9999; visual cylinder length=0.7373221410868707 radius=0.9999
- added link 212, mass 2.3159025717669146; collision cylinder length=0.7373221410868707 radius=0.9999; visual cylinder length=0.7373221410868707 radius=0.9999
- added link 213, mass 2.3159025717669146; collision cylinder length=0.7373221410868707 radius=0.9999; visual cylinder length=0.7373221410868707 radius=0.9999
- added link 214, mass 2.3159025717669146; collision cylinder length=0.7373221410868707 radius=0.9999; visual cylinder length=0.7373221410868707 radius=0.9999
- added link 215, mass 2.3159025717669146; collision cylinder length=0.7373221410868707 radius=0.9999; visual cylinder length=0.7373221410868707 radius=0.9999
- added link 22, mass 2.3159025717669146; collision cylinder length=0.7373221410868707 radius=0.9999; visual cylinder length=0.7373221410868707 radius=0.9999
- added link 23, mass 2.3159025717669146; collision cylinder length=0.7373221410868707 radius=0.9999; visual cylinder length=0.7373221410868707 radius=0.9999
- added link 24, mass 2.3159025717669146; collision cylinder length=0.7373221410868707 radius=0.9999; visual cylinder length=0.7373221410868707 radius=0.9999
- added link 25, mass 2.3159025717669146; collision cylinder length=0.7373221410868707 radius=0.9999; visual cylinder length=0.7373221410868707 radius=0.9999
- added link 27, mass 2.3159025717669146; collision cylinder length=0.7373221410868707 radius=0.9999; visual cylinder length=0.7373221410868707 radius=0.9999
- added link 28, mass 2.3159025717669146; collision cylinder length=0.7373221410868707 radius=0.9999; visual cylinder length=0.7373221410868707 radius=0.9999
- added link 29, mass 2.3159025717669146; collision cylinder length=0.7373221410868707 radius=0.9999; visual cylinder length=0.7373221410868707 radius=0.9999
- link 0: mass 1.6742212661303668 -> 2.3159025717669146; geometry collision cylinder length=0.7373221410868707 radius=0.9999; visual cylinder length=0.7373221410868707 radius=0.9999
Joints:
- added joint 111_to_0: type revolute, parent 0, child 111, origin xyz=0.8429589359258589 0.7886703401700738 0.9999 rpy=24.926035003195217 3.826992907153868 4.104114553209477, axis 1 0 0, limit lower=3.1415 upper=-3.1415 effort=1 velocity=1
- added joint 11_to_0: type revolute, parent 0, child 11, origin xyz=0.8429589359258589 0.7886703401700738 0.9999 rpy=12.463017501597609 3.826992907153868 4.104114553209477, axis 1 0 0, limit lower=3.1415 upper=-3.1415 effort=1 velocity=1
- added joint 16_to_0: type revolute, parent 0, child 16, origin xyz=0.8429589359258589 0.7886703401700738 0.9999 rpy=18.694526252396415 3.826992907153868 4.104114553209477, axis 1 0 0, limit lower=3.1415 upper=-3.1415 effort=1 velocity=1
- added joint 210_to_16: type revolute, parent 16, child 210, origin xyz=0.322992367260043 0.5415013497695964 0.7138715724943219 rpy=27.699172559298894 0.7499782918577459 2.3383200886764004, axis 0 0 1, limit lower=3.1415 upper=-3.1415 effort=1 velocity=1
- added joint 212_to_111: type revolute, parent 111, child 212, origin xyz=0.322992367260043 0.5415013497695964 0.7138715724943219 rpy=11.079669023719557 0.7499782918577459 2.3383200886764004, axis 0 0 1, limit lower=3.1415 upper=-3.1415 effort=1 velocity=1
- added joint 213_to_111: type revolute, parent 111, child 213, origin xyz=0.322992367260043 0.5415013497695964 0.7138715724943219 rpy=16.619503535579334 0.7499782918577459 2.3383200886764004, axis 0 0 1, limit lower=3.1415 upper=-3.1415 effort=1 velocity=1
- added joint 214_to_111: type revolute, parent 111, child 214, origin xyz=0.322992367260043 0.5415013497695964 0.7138715724943219 rpy=22.159338047439114 0.7499782918577459 2.3383200886764004, axis 0 0 1, limit lower=3.1415 upper=-3.1415 effort=1 velocity=1
- added joint 215_to_111: type revolute, parent 111, child 215, origin xyz=0.322992367260043 0.5415013497695964 0.7138715724943219 rpy=27.699172559298894 0.7499782918577459 2.3383200886764004, axis 0 0 1, limit lower=3.1415 upper=-3.1415 effort=1 velocity=1
- added joint 22_to_11: type revolute, parent 11, child 22, origin xyz=0.322992367260043 0.5415013497695964 0.7138715724943219 rpy=11.079669023719557 0.7499782918577459 2.3383200886764004, axis 0 0 1, limit lower=3.1415 upper=-3.1415 effort=1 velocity=1
- added joint 23_to_11: type revolute, parent 11, child 23, origin xyz=0.322992367260043 0.5415013497695964 0.7138715724943219 rpy=16.619503535579334 0.7499782918577459 2.3383200886764004, axis 0 0 1, limit lower=3.1415 upper=-3.1415 effort=1 velocity=1
- added joint 24_to_11: type revolute, parent 11, child 24, origin xyz=0.322992367260043 0.5415013497695964 0.7138715724943219 rpy=22.159338047439114 0.7499782918577459 2.3383200886764004, axis 0 0 1, limit lower=3.1415 upper=-3.1415 effort=1 velocity=1
- added joint 25_to_11: type revolute, parent 11, child 25, origin xyz=0.322992367260043 0.5415013497695964 0.7138715724943219 rpy=27.699172559298894 0.7499782918577459 2.3383200886764004, axis 0 0 1, limit lower=3.1415 upper=-3.1415 effort=1 velocity=1
- added joint 27_to_16: type revolute, parent 16, child 27, origin xyz=0.322992367260043 0.5415013497695964 0.7138715724943219 rpy=11.079669023719557 0.7499782918577459 2.3383200886764004, axis 0 0 1, limit lower=3.1415 upper=-3.1415 effort=1 velocity=1
- added joint 28_to_16: type revolute, parent 16, child 28, origin xyz=0.322992367260043 0.5415013497695964 0.7138715724943219 rpy=16.619503535579334 0.7499782918577459 2.3383200886764004, axis 0 0 1, limit lower=3.1415 upper=-3.1415 effort=1 velocity=1
- added joint 29_to_16: type revolute, parent 16, child 29, origin xyz=0.322992367260043 0.5415013497695964 0.7138715724943219 rpy=22.159338047439114 0.7499782918577459 2.3383200886764004, axis 0 0 1, limit lower=3.1415 upper=-3.1415 effort=1 velocity=1
